File: heart_LED_pcb.kicad_pcb (KiCad board)
At the start: 2 copper layers, 0 parts

Commit message: Updated schematic
Parts:
- added C1: 100nF, Capacitor_SMD:C_0402_1005Metric, F.Cu at (100.5, 113.3)
- added C10: 100nF, Capacitor_SMD:C_0805_2012Metric, F.Cu at (60.7, 154.0)
- added C11: 100nF, Capacitor_SMD:C_0805_2012Metric, F.Cu at (65.2, 138.9)
- added C12: 100nF, Capacitor_SMD:C_0805_2012Metric, F.Cu at (65.2, 142.0)
- added C13: 100nF, Capacitor_SMD:C_0805_2012Metric, F.Cu at (65.2, 145.0)
- added C14: 100nF, Capacitor_SMD:C_0805_2012Metric, F.Cu at (65.2, 148.0)
- added C15: 100nF, Capacitor_SMD:C_0805_2012Metric, F.Cu at (65.2, 151.0)
- added C16: 100nF, Capacitor_SMD:C_0805_2012Metric, F.Cu at (65.2, 154.0)
- added C17: 100nF, Capacitor_SMD:C_0805_2012Metric, F.Cu at (69.6, 138.9)
- added C18: 100nF, Capacitor_SMD:C_0805_2012Metric, F.Cu at (69.6, 142.0)
- added C19: 100nF, Capacitor_SMD:C_0805_2012Metric, F.Cu at (69.6, 145.0)
- added C2: 10uF, Capacitor_SMD:C_0805_2012Metric, F.Cu at (60.7, 138.9)
- added C20: 100nF, Capacitor_SMD:C_0805_2012Metric, F.Cu at (69.6, 148.0)
- added C21: 100nF, Capacitor_SMD:C_0805_2012Metric, F.Cu at (69.6, 151.0)
- added C22: 100nF, Capacitor_SMD:C_0805_2012Metric, F.Cu at (69.6, 154.0)
- added C23: 100nF, Capacitor_SMD:C_0805_2012Metric, F.Cu at (74.0, 138.9)
- added C24: 100nF, Capacitor_SMD:C_0805_2012Metric, F.Cu at (74.0, 142.0)
- added C25: 100nF, Capacitor_SMD:C_0805_2012Metric, F.Cu at (74.0, 145.0)
- added C26: 100nF, Capacitor_SMD:C_0805_2012Metric, F.Cu at (74.0, 148.0)
- added C27: 100nF, Capacitor_SMD:C_0805_2012Metric, F.Cu at (74.0, 151.0)
- added C28: 100nF, Capacitor_SMD:C_0805_2012Metric, F.Cu at (74.0, 154.0)
- added C29: 100nF, Capacitor_SMD:C_0805_2012Metric, F.Cu at (78.5, 138.9)
- added C3: 10uF, Capacitor_SMD:C_0805_2012Metric, F.Cu at (60.7, 142.0)
- added C30: 100nF, Capacitor_SMD:C_0805_2012Metric, F.Cu at (78.5, 142.0)
- added C31: 100nF, Capacitor_SMD:C_0805_2012Metric, F.Cu at (78.5, 145.0)
- added C32: 100nF, Capacitor_SMD:C_0805_2012Metric, F.Cu at (78.5, 148.0)
- added C33: 100nF, Capacitor_SMD:C_0805_2012Metric, F.Cu at (78.5, 151.0)
- added C34: 100nF, Capacitor_SMD:C_0805_2012Metric, F.Cu at (78.5, 154.0)
- added C4: 100nF, Capacitor_SMD:C_0402_1005Metric, F.Cu at (100.5, 115.3)
- added C5: 10uF, Capacitor_SMD:C_0402_1005Metric, F.Cu at (100.5, 117.2)
- added C6: 22uF, Capacitor_Tantalum_SMD:CP_EIA-3216-18_Kemet-A, F.Cu at (100.0, 139.0)
- added C7: 100nF, Capacitor_SMD:C_0805_2012Metric, F.Cu at (60.7, 145.0)
- added C8: 100nF, Capacitor_SMD:C_0805_2012Metric, F.Cu at (60.7, 148.0)
- added C9: 100nF, Capacitor_SMD:C_0805_2012Metric, F.Cu at (60.7, 151.0)
- added D1: WS2812B, LED_SMD:LED_WS2812B_PLCC4_5.0x5.0mm_P3.2mm, F.Cu at (141.7, 122.0)
- added D10: WS2812B, LED_SMD:LED_WS2812B_PLCC4_5.0x5.0mm_P3.2mm, F.Cu at (136.9, 68.2)
- added D11: WS2812B, LED_SMD:LED_WS2812B_PLCC4_5.0x5.0mm_P3.2mm, F.Cu at (144.6, 74.0)
- added D12: WS2812B, LED_SMD:LED_WS2812B_PLCC4_5.0x5.0mm_P3.2mm, F.Cu at (151.4, 82.2)
- added D13: WS2812B, LED_SMD:LED_WS2812B_PLCC4_5.0x5.0mm_P3.2mm, F.Cu at (157.8, 74.5)
- added D14: WS2812B, LED_SMD:LED_WS2812B_PLCC4_5.0x5.0mm_P3.2mm, F.Cu at (165.8, 67.8)
- added D15: WS2812B, LED_SMD:LED_WS2812B_PLCC4_5.0x5.0mm_P3.2mm, F.Cu at (174.2, 66.3)
- added D16: WS2812B, LED_SMD:LED_WS2812B_PLCC4_5.0x5.0mm_P3.2mm, F.Cu at (182.4, 69.7)
- added D17: WS2812B, LED_SMD:LED_WS2812B_PLCC4_5.0x5.0mm_P3.2mm, F.Cu at (187.8, 77.1)
- added D18: WS2812B, LED_SMD:LED_WS2812B_PLCC4_5.0x5.0mm_P3.2mm, F.Cu at (187.3, 85.5)
- added D19: WS2812B, LED_SMD:LED_WS2812B_PLCC4_5.0x5.0mm_P3.2mm, F.Cu at (185.2, 92.8)
- added D2: WS2812B, LED_SMD:LED_WS2812B_PLCC4_5.0x5.0mm_P3.2mm, F.Cu at (134.3, 115.7)
- added D20: WS2812B, LED_SMD:LED_WS2812B_PLCC4_5.0x5.0mm_P3.2mm, F.Cu at (180.6, 100.3)
- added D21: WS2812B, LED_SMD:LED_WS2812B_PLCC4_5.0x5.0mm_P3.2mm, F.Cu at (174.5, 107.2)
- added D22: WS2812B, LED_SMD:LED_WS2812B_PLCC4_5.0x5.0mm_P3.2mm, F.Cu at (167.4, 114.2)
- added D23: WS2812B, LED_SMD:LED_WS2812B_PLCC4_5.0x5.0mm_P3.2mm, F.Cu at (160.6, 121.3)
- added D24: WS2812B, LED_SMD:LED_WS2812B_PLCC4_5.0x5.0mm_P3.2mm, F.Cu at (95.0, 127.5)
- added D25: WS2812B, LED_SMD:LED_WS2812B_PLCC4_5.0x5.0mm_P3.2mm, F.Cu at (95.0, 134.1)
- added D3: WS2812B, LED_SMD:LED_WS2812B_PLCC4_5.0x5.0mm_P3.2mm, F.Cu at (128.2, 109.2)
- added D4: WS2812B, LED_SMD:LED_WS2812B_PLCC4_5.0x5.0mm_P3.2mm, F.Cu at (122.2, 102.2)
- added D5: WS2812B, LED_SMD:LED_WS2812B_PLCC4_5.0x5.0mm_P3.2mm, F.Cu at (117.2, 94.8)
- added D6: WS2812B, LED_SMD:LED_WS2812B_PLCC4_5.0x5.0mm_P3.2mm, F.Cu at (114.3, 87.0)
- added D7: WS2812B, LED_SMD:LED_WS2812B_PLCC4_5.0x5.0mm_P3.2mm, F.Cu at (114.8, 78.7)
- added D8: WS2812B, LED_SMD:LED_WS2812B_PLCC4_5.0x5.0mm_P3.2mm, F.Cu at (119.5, 71.0)
- added D9: WS2812B, LED_SMD:LED_WS2812B_PLCC4_5.0x5.0mm_P3.2mm, F.Cu at (127.9, 66.6)
- added J1: USB_C_2.0_16P, Connector_USB:USB_C_Receptacle_G-Switch_GT-USB-7010ASV, F.Cu at (151.1, 129.7)
- added R1: 5.1k, Resistor_SMD:R_0603_1608Metric, F.Cu at (99.1, 146.4)
- added R2: 5.1k, Resistor_SMD:R_0603_1608Metric, F.Cu at (99.1, 148.9)
- added R3: 10k, Resistor_SMD:R_0402_1005Metric, F.Cu at (100.5, 105.3)
- added R4: 10k, Resistor_SMD:R_0402_1005Metric, F.Cu at (100.5, 107.3)
- added R5: 10k, Resistor_SMD:R_0402_1005Metric, F.Cu at (100.5, 109.3)
- added R6: 10k, Resistor_SMD:R_0402_1005Metric, F.Cu at (100.5, 111.3)
- added SW1: EN, Button_Switch_SMD:SW_Push_SPST_NO_Alps_SKRK, F.Cu at (93.8, 139.7)
- added SW2: BOOT, Button_Switch_SMD:SW_Push_SPST_NO_Alps_SKRK, F.Cu at (93.8, 144.1)
- added SW3: MODE, Button_Switch_SMD:SW_Push_SPST_NO_Alps_SKRK, F.Cu at (93.8, 148.6)
- added SW4: LED_MODUS, Button_Switch_SMD:SW_Push_SPST_NO_Alps_SKRK, F.Cu at (93.8, 153.0)
- added U1: ESP32-C3, Package_DFN_QFN:QFN-32-1EP_5x5mm_P0.5mm_EP3.45x3.45mm, F.Cu at (70.5, 80.2)
- added U2: AMS1117-3.3, Package_TO_SOT_SMD:SOT-223-3_TabPin2, F.Cu at (70.6, 89.8)
- added Y1: 40 MHz, Crystal:Crystal_SMD_TXC_7M-4Pin_3.2x2.5mm, F.Cu at (99.8, 142.9)
Other:
- board outline added: 85.8 x 78.4 mm
- copper layers 2 -> 4
