File: heart_LED_pcb.kicad_sch (KiCad schematic)
At the start: 6 parts, among them J1 USB_C_2.0_16P, U1 ESP32-C3, U2 AMS1117-3.3

Commit message: Updated schematic
Parts:
- added C1: 100nF, Capacitor_SMD:CP_Elec_CAP-XX_DMF3Zxxxxxxxx3D, symbol Device:C_Small
- added C2, C3: 10uF, symbol Device:C_Small
- added C4: 100nF, symbol Device:C_Small
- added C5: 100nF, Capacitor_SMD:C_0402_1005Metric, symbol Device:C
- added C6: 22uF, Capacitor_Tantalum_SMD:CP_EIA-3216-18_Kemet-A, symbol Device:C_Polarized
- added C7: 100nF, Capacitor_SMD:C_0201_0603Metric, symbol Device:C_Small
- added R3, R4, R5: 10k, symbol Device:R_Small
- added SW1: EN, symbol Switch:SW_Push
- added SW2: BOOT, symbol Switch:SW_Push
- added SW3: MODE, symbol Switch:SW_Push
- added Y1: 40 MHz, Crystal:Crystal_SMD_TXC_7M-4Pin_3.2x2.5mm, symbol Device:Crystal_GND24_Small
Connections:
- net +5V: now also D1.1 (VDD), C5.1, C7.1
- net GND: now also D1.3 (VSS), C1.2, C2.2, C3.2, C4.1, C5.2, C6.2, C7.2, SW1.1, SW2.1, SW3.1, Y1.2, Y1.4
- net +3.3V: now reaches U1.11 (VDD3P3_RTC)
- net +3.3V: now also U1.17 (VDD3P3_CPU), U1.2 (VDD3P3), U1.3 (VDD3P3), U1.31 (VDDA), U1.32 (VDDA), U2.2 (VO), C1.1, C6.1, R3.1, R4.1, R5.1
- net LED_MODUS: now reaches U1.14 (GPIO8)
- net BOOT: now reaches U1.15 (GPIO9/BOOT)
- net BOOT: now also R4.2, SW2.2
- net LED_PWM: now reaches U1.16 (GPIO10)
- net LED_PWM: now also D1.4 (DIN), R5.2, SW3.2
- net XTAL_P: now reaches U1.29 (XTAL_N)
- net XTAL_P: now also C3.1, Y1.1
- net XTAL_N: now reaches U1.30 (XTAL_P)
- net XTAL_N: now also C2.1, Y1.3
- net EN: now reaches U1.7 (CHIP_EN)
- net EN: now also C4.2, R3.2, SW1.2
- no-connect marks 2 -> 20
Other:
- added sheet ESP32-C3 (ESP32-C3.kicad_sch)
- added sheet LDO 5V -> 3V3 (LDO_ESP32_C3.kicad_sch)
- added sheet USB_C_2.0 (USB_C_2.0.kicad_sch)
- moved on the sheet: D1, J1, U1, U2

Commit message: Updated schematic
Parts:
- added C10, C11, C12, C13, C14, C15, C16, C17, C18, C19, C20, C21, C8, C9: 100nF, Capacitor_SMD:C_0201_0603Metric, symbol Device:C_Small
- added D10, D11, D12, D13, D14, D15, D2, D3, D4, D5, D6, D7, D8, D9: WS2812B, LED_SMD:LED_WS2812B_PLCC4_5.0x5.0mm_P3.2mm, symbol LED:WS2812B
- added R6: 10k, Resistor_SMD:R_0402_1005Metric, symbol Device:R_Small
- added SW4: LED_MODUS, symbol Switch:SW_Push
- R3, R4, R5: footprint (none) -> Resistor_SMD:R_0402_1005Metric
Connections:
- net +3.3V: now also R6.1
- net +5V: now also C10.1, C11.1, C12.1, C13.1, C14.1, C15.1, C16.1, C17.1, C18.1, C19.1, C20.1, C21.1, C8.1, C9.1, D10.1 (VDD), D11.1 (VDD), D12.1 (VDD), D13.1 (VDD), D14.1 (VDD), D15.1 (VDD), D2.1 (VDD), D3.1 (VDD), D4.1 (VDD), D5.1 (VDD), D6.1 (VDD), D7.1 (VDD), D8.1 (VDD), D9.1 (VDD)
- net GND: now also C10.2, C11.2, C12.2, C13.2, C14.2, C15.2, C16.2, C17.2, C18.2, C19.2, C20.2, C21.2, C8.2, C9.2, D10.3 (VSS), D11.3 (VSS), D12.3 (VSS), D13.3 (VSS), D14.3 (VSS), D15.2 (DOUT), D15.3 (VSS), D2.3 (VSS), D3.3 (VSS), D4.3 (VSS), D5.3 (VSS), D6.3 (VSS), D7.3 (VSS), D8.3 (VSS), D9.3 (VSS), SW4.1
- net LED_MODUS: now also R6.2, SW4.2
- net at D1.2 (DOUT): now also D2.4 (DIN)
- new net: D6.2 (DOUT), D7.4 (DIN)
- new net: D14.2 (DOUT), D15.4 (DIN)
- new net: D7.2 (DOUT), D8.4 (DIN)
- new net: D13.2 (DOUT), D14.4 (DIN)
- new net: D12.2 (DOUT), D13.4 (DIN)
- new net: D10.4 (DIN), D9.2 (DOUT)
- new net: D4.2 (DOUT), D5.4 (DIN)
- new net: D3.2 (DOUT), D4.4 (DIN)
- new net: D2.2 (DOUT), D3.4 (DIN)
- new net: D8.2 (DOUT), D9.4 (DIN)
- new net: D11.2 (DOUT), D12.4 (DIN)
- new net LED0: D5.2 (DOUT), D6.4 (DIN)
- new net LED1: D10.2 (DOUT), D11.4 (DIN)
Other:
- moved on the sheet: C7, D1

Commit message: Updated schematic
Parts:
- added C22, C23, C24, C25, C26, C27, C28, C29, C30, C31, C32, C33, C34: 100nF, Capacitor_SMD:C_0805_2012Metric, symbol Device:C_Small
- added D16, D17, D18, D19, D20, D21, D22, D23, D24, D25: WS2812B, LED_SMD:LED_WS2812B_PLCC4_5.0x5.0mm_P3.2mm, symbol LED:WS2812B
- C1: footprint Capacitor_SMD:CP_Elec_CAP-XX_DMF3Zxxxxxxxx3D -> Capacitor_SMD:C_0402_1005Metric
- C10, C11, C12, C13, C14, C15, C16, C17, C18, C19, C20, C21, C7, C8, C9: footprint Capacitor_SMD:C_0201_0603Metric -> Capacitor_SMD:C_0805_2012Metric
- C2, C3: footprint (none) -> Capacitor_SMD:C_0805_2012Metric
- C4: footprint (none) -> Capacitor_SMD:C_0402_1005Metric
- C5: value 100nF -> 10uF
- SW1, SW2, SW3, SW4: footprint (none) -> Button_Switch_SMD:SW_Push_SPST_NO_Alps_SKRK
Connections:
- net +3.3V: now also C32.1, C33.1, C34.1
- net +5V: now also C22.1, C23.1, C24.1, C25.1, C26.1, C27.1, C28.1, C29.1, C30.1, C31.1, D16.1 (VDD), D17.1 (VDD), D18.1 (VDD), D19.1 (VDD), D20.1 (VDD), D21.1 (VDD), D22.1 (VDD), D23.1 (VDD), D24.1 (VDD), D25.1 (VDD)
- net GND: now also C22.2, C23.2, C24.2, C25.2, C26.2, C27.2, C28.2, C29.2, C30.2, C31.2, C32.2, C33.2, C34.2, D16.3 (VSS), D17.3 (VSS), D18.3 (VSS), D19.3 (VSS), D20.3 (VSS), D21.3 (VSS), D22.3 (VSS), D23.3 (VSS), D24.3 (VSS), D25.3 (VSS); no longer D15.2 (DOUT)
- new net: D22.2 (DOUT), D23.4 (DIN)
- new net: D21.2 (DOUT), D22.4 (DIN)
- new net: D19.2 (DOUT), D20.4 (DIN)
- new net: D17.2 (DOUT), D18.4 (DIN)
- new net: D16.2 (DOUT), D17.4 (DIN)
- new net: D24.2 (DOUT), D25.4 (DIN)
- new net: D23.2 (DOUT), D24.4 (DIN)
- new net: D18.2 (DOUT), D19.4 (DIN)
- new net LED2: D15.2 (DOUT), D16.4 (DIN)
- new net LED3: D20.2 (DOUT), D21.4 (DIN)
- no-connect marks 20 -> 21
Other:
- removed sheet ESP32-C3
- removed sheet LDO 5V -> 3V3
- removed sheet USB_C_2.0
- title: (none) -> ESP32-Heart-LED-PCB
- moved on the sheet: C1, C10, C11, C12, C13, C14, C15, C16, C17, C18, C19, C2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

Commit message: Updated schematic
Parts:
- removed C30, C31: 100nF, Capacitor_SMD:C_0805_2012Metric, symbol Device:C_Small
- removed D24, D25: WS2812B, LED_SMD:LED_WS2812B_PLCC4_5.0x5.0mm_P3.2mm, symbol LED:WS2812B
- removed R5: 10k, Resistor_SMD:R_0402_1005Metric, symbol Device:R_Small
- removed SW3: MODE, Button_Switch_SMD:SW_Push_SPST_NO_Alps_SKRK, symbol Switch:SW_Push
- added C35: 100nF, Capacitor_SMD:C_0402_1005Metric, symbol Device:C_Small
- renumbered SW4 to SW3
Connections:
- net +5V: now also C35.1
- net GND: now also C35.2
- net LED_MODUS: now also U1.16 (GPIO10); no longer U1.14 (GPIO8)
- net LED_PWM: no longer U1.16 (GPIO10)
- no-connect marks 21 -> 22
